Commit message: Added support for Gazebo

File: src/xerbo_description/src/urdf/create_base.urdf.xacro (robot description, xacro)
@@ -4,23 +4,23 @@
   <xacro:macro name="create_wheel" params="prefix y_offset wheel_radius wheel_width">
     <link name="${prefix}_wheel_link">
-    <inertial>
-      <origin xyz="0 0 0" />
-      <mass value="0.01" />
-      <inertia ixx="0.001" ixy="0.0" ixz="0.0" iyy="0.001" iyz="0.0" izz="0.001" />
-    </inertial>
-    <visual>
-      <origin xyz="0 0 0" rpy="0 ${PI/2} ${PI/2}" />
-      <geometry>
-        <cylinder radius="${wheel_radius}" length="${wheel_width}" />
-      </geometry>
-    </visual>
-    <collision>
-      <origin xyz="0 0 0" rpy="0 ${PI/2} ${PI/2}" />
-      <geometry>
-        <cylinder radius="${wheel_radius}" length="${wheel_width}" />
-      </geometry>
-    </collision>
+      <inertial>
+        <origin xyz="0 0 0" />
+        <mass value="0.01" />
+        <inertia ixx="0.001" ixy="0.0" ixz="0.0" iyy="0.001" iyz="0.0" izz="0.001" />
+      </inertial>
+      <visual>
+        <origin xyz="0 0 0" rpy="0 ${PI/2} ${PI/2}" />
+        <geometry>
+          <cylinder radius="${wheel_radius}" length="${wheel_width}" />
+        </geometry>
+      </visual>
+      <collision>
+        <origin xyz="0 0 0" rpy="0 ${PI/2} ${PI/2}" />
+        <geometry>
+          <cylinder radius="${wheel_radius}" length="${wheel_width}" />
+        </geometry>
+      </collision>
     </link>
-   <joint name="${prefix}_wheel_joint" type="continuous">
+    <joint name="${prefix}_wheel_joint" type="continuous">
       <origin xyz="0 ${y_offset} 0.015" rpy="0 0 0" />
       <parent link="base_link" />
@@ -32,71 +32,71 @@
     <xacro:include filename="$(find xerbo_description)/src/urdf/create_base_gazebo.urdf.xacro" />
     <link name="base_footprint">
-    <visual>
-      <origin xyz="0 0 0" rpy="0 0 0" />
-      <geometry>
-        <box size="0.001 0.001 0.001" />
-      </geometry>
-      <material name="Green" />
-    </visual>
-    <collision>
-      <origin xyz="0 0 0.017" rpy="0 0 0" />
-      <geometry>
-        <box size="0.001 0.001 0.001" />
-      </geometry>
-    </collision>
+      <visual>
+        <origin xyz="0 0 0" rpy="0 0 0" />
+        <geometry>
+          <box size="0.001 0.001 0.001" />
+        </geometry>
+        <material name="Green" />
+      </visual>
+      <collision>
+        <origin xyz="0 0 0.017" rpy="0 0 0" />
+        <geometry>
+          <box size="0.001 0.001 0.001" />
+        </geometry>
+      </collision>
     </link>
     <link name="base_link">
-    <inertial>
-      <mass value="2" />
-      <origin xyz="0 0 0.0" />
-      <inertia ixx="0.01" ixy="0.0" ixz="0.0" iyy="0.01" iyz="0.0" izz="0.5" />
-    </inertial>
-    <visual>
-      <origin xyz=" 0 0 0.0308" rpy="0 0 0" />
-      <geometry>
-        <xacro:insert_block name="mesh" />
-      </geometry>
-    </visual>
-    <collision>
-      <origin xyz="0.0 0.0 0.0308" rpy="0 0 0" />
-      <geometry>
-        <cylinder length="0.0611632" radius="0.16495" />
-      </geometry>
-    </collision>
+      <inertial>
+        <mass value="2" />
+        <origin xyz="0 0 0.0" />
+        <inertia ixx="0.01" ixy="0.0" ixz="0.0" iyy="0.01" iyz="0.0" izz="0.5" />
+      </inertial>
+      <visual>
+        <origin xyz=" 0 0 0.0308" rpy="0 0 0" />
+        <geometry>
+          <xacro:insert_block name="mesh" />
+        </geometry>
+      </visual>
+      <collision>
+        <origin xyz="0.0 0.0 0.0308" rpy="0 0 0" />
+        <geometry>
+          <cylinder length="0.0611632" radius="0.16495" />
+        </geometry>
+      </collision>
     </link>
     <link name="wall_sensor_link">
-    <inertial>
-      <mass value="0.01" />
-      <origin xyz="0 0 0" />
-      <inertia ixx="0.001" ixy="0.0" ixz="0.0" iyy="0.001" iyz="0.0" izz="0.001" />
-    </inertial>
+      <inertial>
+        <mass value="0.01" />
+        <origin xyz="0 0 0" />
+        <inertia ixx="0.001" ixy="0.0" ixz="0.0" iyy="0.001" iyz="0.0" izz="0.001" />
+      </inertial>
     </link>
     <link name="left_cliff_sensor_link">
-    <inertial>
-      <mass value="0.01" />
-      <origin xyz="0 0 0" />
-      <inertia ixx="0.001" ixy="0.0" ixz="0.0" iyy="0.001" iyz="0.0" izz="0.001" />
-    </inertial>
+      <inertial>
+        <mass value="0.01" />
+        <origin xyz="0 0 0" />
+        <inertia ixx="0.001" ixy="0.0" ixz="0.0" iyy="0.001" iyz="0.0" izz="0.001" />
+      </inertial>
     </link>
     <link name="right_cliff_sensor_link">
-    <inertial>
-      <mass value="0.01" />
-      <origin xyz="0 0 0" />
-      <inertia ixx="0.001" ixy="0.0" ixz="0.0" iyy="0.001" iyz="0.0" izz="0.001" />
-    </inertial>
+      <inertial>
+        <mass value="0.01" />
+        <origin xyz="0 0 0" />
+        <inertia ixx="0.001" ixy="0.0" ixz="0.0" iyy="0.001" iyz="0.0" izz="0.001" />
+      </inertial>
     </link>
     <link name="leftfront_cliff_sensor_link">
-    <inertial>
-      <mass value="0.01" />
-      <origin xyz="0 0 0" />
-      <inertia ixx="1.0" ixy="0.0" ixz="0.0" iyy="0.01" iyz="0.0" izz="0.01" />
-    </inertial>
+      <inertial>
+        <mass value="0.01" />
+        <origin xyz="0 0 0" />
+        <inertia ixx="1.0" ixy="0.0" ixz="0.0" iyy="0.01" iyz="0.0" izz="0.01" />
+      </inertial>
     </link>
     <link name="rightfront_cliff_sensor_link">
-    <inertial>
-      <mass value="0.01" />
-      <origin xyz="0 0 0" />
-      <inertia ixx="0.001" ixy="0.0" ixz="0.0" iyy="0.001" iyz="0.0" izz="0.001" />
-    </inertial>
+      <inertial>
+        <mass value="0.01" />
+        <origin xyz="0 0 0" />
+        <inertia ixx="0.001" ixy="0.0" ixz="0.0" iyy="0.001" iyz="0.0" izz="0.001" />
+      </inertial>
     </link>
     <joint name="base_footprint_joint" type="fixed">
@@ -132,48 +132,22 @@
     <xacro:create_wheel prefix="left" y_offset="${wheel_separation / 2}" wheel_radius="${wheel_radius}" wheel_width="${wheel_width}"/>
     <xacro:create_wheel prefix="right" y_offset="${wheel_separation / -2}" wheel_radius="${wheel_radius}" wheel_width="${wheel_width}"/>
-    <!--<link name="rear_wheel_link">
-    <inertial>
-      <origin xyz="0 0 0"/>
-      <mass value="0.001" />
-      <inertia ixx="0.0001" ixy="0.0" ixz="0.0"
-        iyy="0.0001" iyz="0.0" izz="0.0001" />
-    </inertial>
-    <visual>
-      <origin xyz="0 0 0" rpy="0 ${PI/2} ${PI/2}"/>
-      <geometry>
-        <sphere radius="0.015" />
-      </geometry>
-    </visual>
-    <collision>
-      <origin xyz="0 0 0" rpy="0 ${PI/2} ${PI/2}" />
-      <geometry>
-        <sphere radius="0.015" />
-      </geometry>
-    </collision>
-    </link>
-    <joint name="rear_castor_joint" type="fixed">
-      <origin xyz="-0.13 0 0.0" rpy="0 0 0"/>
-      <parent link="base_link"/>
-      <child link="rear_wheel_link"/>
-      <axis xyz="0 1 0"/>
-    </joint>-->
     <link name="front_wheel_link">
-    <inertial>
-      <origin xyz="0 0 0" />
-      <mass value="0.01" />
-      <inertia ixx="0.001" ixy="0.0" ixz="0.0" iyy="0.001" iyz="0.0" izz="0.001" />
-    </inertial>
-    <visual>
-      <origin xyz="0 0 0" rpy="0 ${PI/2} ${PI/2}" />
-      <geometry>
-        <sphere radius="0.018" />
-      </geometry>
-    </visual>
-    <collision>
-      <origin xyz="0 0 0" rpy="0 ${PI/2} ${PI/2}" />
-      <geometry>
-        <sphere radius="0.018" />
-      </geometry>
-    </collision>
+      <inertial>
+        <origin xyz="0 0 0" />
+        <mass value="0.01" />
+        <inertia ixx="0.001" ixy="0.0" ixz="0.0" iyy="0.001" iyz="0.0" izz="0.001" />
+      </inertial>
+      <visual>
+        <origin xyz="0 0 0" rpy="0 ${PI/2} ${PI/2}" />
+        <geometry>
+          <sphere radius="0.018" />
+        </geometry>
+      </visual>
+      <collision>
+        <origin xyz="0 0 0" rpy="0 ${PI/2} ${PI/2}" />
+        <geometry>
+          <sphere radius="0.018" />
+        </geometry>
+      </collision>
     </link>
     <!-- fixed because there's no transmission -->
@@ -191,9 +165,9 @@
     </joint>
     <link name="gyro_link">
-    <inertial>
-      <mass value="0.001" />
-      <origin xyz="0 0 0" rpy="0 0 0" />
-      <inertia ixx="0.0001" ixy="0" ixz="0" iyy="0.000001" iyz="0" izz="0.0001" />
-    </inertial>
+      <inertial>
+        <mass value="0.001" />
+        <origin xyz="0 0 0" rpy="0 0 0" />
+        <inertia ixx="0.0001" ixy="0" ixz="0" iyy="0.000001" iyz="0" izz="0.0001" />
+      </inertial>
     </link>
     <!-- Simulation sensors -->

File: src/xerbo_description/src/urdf/create_base_gazebo.urdf.xacro (robot description, xacro)
@@ -4,27 +4,28 @@
     <gazebo>
       <plugin name="differential_drive_controller" filename="libgazebo_ros_diff_drive.so">
-        <alwaysOn>true</alwaysOn>
-        <updateRate>${diffdrive_update_rate}</updateRate>
-        <leftJoint>left_wheel_joint</leftJoint>
-        <rightJoint>right_wheel_joint</rightJoint>
-        <wheelSeparation>${wheel_separation}</wheelSeparation>
-        <wheelDiameter>${wheel_radius * 2}</wheelDiameter>
-        <wheelTorque>${wheel_torque}</wheelTorque>
-        <!--wheelAcceleration>${wheel_accel}</wheelAcceleration-->
-        <commandTopic>cmd_vel</commandTopic>
-        <odometryTopic>odom</odometryTopic>
-        <odometryFrame>odom</odometryFrame>
-        <robotBaseFrame>base_footprint</robotBaseFrame>
+        <always_on>true</always_on>
+        <update_rate>${diffdrive_update_rate}</update_rate>
+        <left_joint>left_wheel_joint</left_joint>
+        <right_joint>right_wheel_joint</right_joint>
+        <wheel_separation>${wheel_separation}</wheel_separation>
+        <wheel_diameter>${wheel_radius * 2}</wheel_diameter>
+        <wheel_torque>${wheel_torque}</wheel_torque>
+        <command_topic>cmd_vel</command_topic>
+        <odometry_topic>odom</odometry_topic>
+        <odometry_frame>odom</odometry_frame>
+        <robot_base_frame>base_footprint</robot_base_frame>
+        <publish_odom>true</publish_odom>
+        <publish_odom_tf>true</publish_odom_tf>
+        <publish_wheel_tf>true</publish_wheel_tf>
       </plugin>
       <plugin name="p3d_base_controller" filename="libgazebo_ros_p3d.so">
-        <alwaysOn>true</alwaysOn>
-        <updateRate>100.0</updateRate>
-        <bodyName>base_link</bodyName>
-        <topicName>simple_controller/absolute_position</topicName>
-        <gaussianNoise>0</gaussianNoise>
-        <frameName>map</frameName>
-        <xyzOffsets>0 0 0</xyzOffsets>
-        <rpyOffsets>0 0 0</rpyOffsets>
-        <!--<interface:position name="p3d_base_position"/>-->
+        <always_on>true</always_on>
+        <update_rate>100.0</update_rate>
+        <body_name>base_link</body_name>
+        <topic_name>simple_controller/absolute_position</topic_name>
+        <gaussian_noise>0</gaussian_noise>
+        <frame_name>map</frame_name>
+        <xyz_offsets>0 0 0</xyz_offsets>
+        <rpy_offsets>0 0 0</rpy_offsets>
       </plugin>
     </gazebo>
@@ -34,6 +35,6 @@
       <kp>1000000.0</kp>
       <kd>100.0</kd>
-      <minDepth>0.001</minDepth>
-      <maxVel>1.0</maxVel>
+      <min_depth>0.001</min_depth>
+      <max_vel>1.0</max_vel>
     </gazebo>
     <gazebo reference="right_wheel_link">
@@ -42,6 +43,6 @@
       <kp>1000000.0</kp>
       <kd>100.0</kd>
-      <minDepth>0.001</minDepth>
-      <maxVel>1.0</maxVel>
+      <min_depth>0.001</min_depth>
+      <max_vel>1.0</max_vel>
     </gazebo>
     <gazebo reference="rear_wheel_link">
@@ -50,6 +51,6 @@
       <kp>1000000.0</kp>
       <kd>100.0</kd>
-      <minDepth>0.001</minDepth>
-      <maxVel>1.0</maxVel>
+      <min_depth>0.001</min_depth>
+      <max_vel>1.0</max_vel>
     </gazebo>
     <gazebo reference="front_wheel_link">
@@ -58,20 +59,27 @@
       <kp>1000000.0</kp>
       <kd>100.0</kd>
-      <minDepth>0.001</minDepth>
-      <maxVel>1.0</maxVel>
+      <min_depth>0.001</min_depth>
+      <max_vel>1.0</max_vel>
     </gazebo>
   </xacro:macro>
   <xacro:macro name="sim_imu">
     <gazebo>
-      <plugin name="imu_controller" filename="libgazebo_ros_imu.so">
-        <alwaysOn>true</alwaysOn>
-        <updateRate>30</updateRate>
-        <bodyName>gyro_link</bodyName>
-        <topicName>imu/data</topicName>
-        <serviceName>imu/is_calibrated</serviceName>
-        <gaussianNoise>${0.0017*0.0017}</gaussianNoise>
-        <xyzOffsets>0 0 0</xyzOffsets>
-        <rpyOffsets>0 0 0</rpyOffsets>
-      </plugin>
+      <sensor name="imu_sensor" type="imu">
+        <always_on>true</always_on>
+        <update_rate>100</update_rate>
+        <visualize>true</visualize>
+        <topic>__default_topic__</topic>
+        <plugin filename="libgazebo_ros_imu_sensor.so" name="imu_plugin">
+          <topic_name>imu_qq</topic_name>
+          <body_name>gyro_link</body_name>
+          <update_rate_hz>10.0</update_rate_hz>
+          <gaussian_noise>${0.0017*0.0017}</gaussian_noise>
+          <xyz_offset>0 0 0</xyz_offset>
+          <rpy_offset>0 0 0</rpy_offset>
+          <frame_name>imu_link</frame_name>
+          <initial_orientation_as_reference>false</initial_orientation_as_reference>
+        </plugin>
+        <pose>0 0 0 0 0 0</pose>
+      </sensor>
     </gazebo>
   </xacro:macro>

File: src/xerbo_description/src/urdf/xerbo.urdf.xacro (robot description, xacro)
@@ -1,7 +1,18 @@
 <?xml version="1.0" ?>
 <robot name="xerbo" xmlns:xacro="http://ros.org/wiki/xacro">
+  <!-- Define intertial property macros  -->
+  <xacro:macro name="box_inertia" params="m w h d">
+    <inertial>
+      <origin xyz="0 0 0" rpy="${pi/2} 0 ${pi/2}"/>
+      <mass value="${m}"/>
+      <inertia ixx="${(m/12) * (h*h + d*d)}" ixy="0.0" ixz="0.0" iyy="${(m/12) * (w*w + d*d)}" iyz="0.0" izz="${(m/12) * (w*w + h*h)}"/>
+    </inertial>
+  </xacro:macro>
   <xacro:include filename="$(find xerbo_description)/src/urdf/create_base.urdf.xacro" />
   <xacro:create_base wheel_separation="0.235" base_diameter="0.3485">
-    <mesh filename="package://xerbo_description/src/meshes/xerbo.dae" />
+    <!-- "file://" syntax is compatible with both RVIZ and Gazebo -->
+    <mesh filename="file://$(find xerbo_description)/src/meshes/xerbo.dae" />
   </xacro:create_base>
+  <xacro:include filename="$(find xerbo_description)/src/urdf/imu_link.urdf.xacro" />
+  <xacro:create_imu connected_to="base_link" />
 </robot>
