Commit message: Moved /src subfolders up to root

File: src/xerbo_description/urdf/create_base.urdf.xacro (robot description, xacro)
@@ -30,5 +30,5 @@
   </xacro:macro>
   <xacro:macro name="create_base" params="diffdrive_update_rate:=40 wheel_separation wheel_radius:=0.036 wheel_width:=0.024 wheel_torque:=1.0 wheel_accel:=1.8 mass_kg:=3.5 base_diameter *mesh">
-    <xacro:include filename="$(find xerbo_description)/src/urdf/create_base_gazebo.urdf.xacro" />
+    <xacro:include filename="$(find xerbo_description)/urdf/create_base_gazebo.urdf.xacro" />
     <link name="base_footprint">
       <visual>

File: src/xerbo_description/urdf/xerbo.urdf.xacro (robot description, xacro)
@@ -9,10 +9,8 @@
     </inertial>
   </xacro:macro>
-  <xacro:include filename="$(find xerbo_description)/src/urdf/create_base.urdf.xacro" />
+  <xacro:include filename="$(find xerbo_description)/urdf/create_base.urdf.xacro" />
   <xacro:create_base wheel_separation="0.235" base_diameter="0.3485">
     <!-- "file://" syntax is compatible with both RVIZ and Gazebo -->
-    <mesh filename="file://$(find xerbo_description)/src/meshes/xerbo.dae" />
+    <mesh filename="file://$(find xerbo_description)/meshes/xerbo.dae" />
   </xacro:create_base>
-  <xacro:include filename="$(find xerbo_description)/src/urdf/imu_link.urdf.xacro" />
-  <xacro:create_imu connected_to="base_link" />
 </robot>

Commit message: Added separate IMU from base URDF

File: src/xerbo_description/urdf/create_base.urdf.xacro (robot description, xacro)
@@ -175,5 +175,4 @@
     <xacro:sim_create_wall_sensor/>
     <xacro:sim_create_cliff_sensors/>
-    <xacro:sim_imu/>
   </xacro:macro>
 </robot>

File: src/xerbo_description/urdf/create_base_gazebo.urdf.xacro (robot description, xacro)
@@ -15,7 +15,9 @@
         <odometry_frame>odom</odometry_frame>
         <robot_base_frame>base_footprint</robot_base_frame>
+        <!--
         <publish_odom>true</publish_odom>
         <publish_odom_tf>true</publish_odom_tf>
         <publish_wheel_tf>true</publish_wheel_tf>
+        -->
       </plugin>
       <plugin name="p3d_base_controller" filename="libgazebo_ros_p3d.so">
@@ -61,25 +63,4 @@
       <min_depth>0.001</min_depth>
       <max_vel>1.0</max_vel>
-    </gazebo>
-  </xacro:macro>
-  <xacro:macro name="sim_imu">
-    <gazebo>
-      <sensor name="imu_sensor" type="imu">
-        <always_on>true</always_on>
-        <update_rate>100</update_rate>
-        <visualize>true</visualize>
-        <topic>__default_topic__</topic>
-        <plugin filename="libgazebo_ros_imu_sensor.so" name="imu_plugin">
-          <topic_name>imu_qq</topic_name>
-          <body_name>gyro_link</body_name>
-          <update_rate_hz>10.0</update_rate_hz>
-          <gaussian_noise>${0.0017*0.0017}</gaussian_noise>
-          <xyz_offset>0 0 0</xyz_offset>
-          <rpy_offset>0 0 0</rpy_offset>
-          <frame_name>imu_link</frame_name>
-          <initial_orientation_as_reference>false</initial_orientation_as_reference>
-        </plugin>
-        <pose>0 0 0 0 0 0</pose>
-      </sensor>
     </gazebo>
   </xacro:macro>

File: src/xerbo_description/urdf/xerbo.urdf.xacro (robot description, xacro)
@@ -14,3 +14,5 @@
     <mesh filename="file://$(find xerbo_description)/meshes/xerbo.dae" />
   </xacro:create_base>
+  <xacro:include filename="$(find xerbo_description)/urdf/imu_link.urdf.xacro" />
+  <xacro:create_imu connected_to="base_link" />
 </robot>
