Commit message: Refactored URDF for clarity and to fix link issue in simulator

File: src/xerbo_description/urdf/imu.gazebo.urdf.xacro (robot description, xacro)
@@ -1,3 +1,3 @@
-<?xml version="1.0" ?>
+<?xml version="1.0"?>
 <robot xmlns:xacro="http://ros.org/wiki/xacro">
   <gazebo reference="imu_link">
@@ -13,8 +13,8 @@
       <update_rate>100</update_rate>
       <visualize>true</visualize>
-      <imu>
-        <angular_velocity>
-          <x>
-            <noise type="gaussian">
+     <imu>
+     	<angular_velocity>
+     	  <x>
+     	    <noise type="gaussian">
               <mean>0.0</mean>
               <stddev>2e-4</stddev>

File: src/xerbo_description/urdf/xerbo.urdf.xacro (robot description, xacro)
@@ -1,5 +1,4 @@
-<?xml version="1.0" ?>
+<?xml version="1.0"?>
 <robot name="xerbo" xmlns:xacro="http://ros.org/wiki/xacro">
-  <!-- Define intertial property macros  -->
   <xacro:macro name="box_inertia" params="m w h d">
     <inertial>
@@ -9,10 +8,6 @@
     </inertial>
   </xacro:macro>
-  <xacro:include filename="$(find xerbo_description)/urdf/create_base.urdf.xacro" />
-  <xacro:create_base wheel_separation="0.235" base_diameter="0.3485">
-    <!-- "file://" syntax is compatible with both RVIZ and Gazebo -->
-    <mesh filename="file://$(find xerbo_description)/meshes/xerbo.dae" />
-  </xacro:create_base>
-  <xacro:include filename="$(find xerbo_description)/urdf/create_imu.urdf.xacro" />
-  <xacro:create_imu connected_to="base_link" />
+  <xacro:include filename="$(find xerbo_description)/urdf/base.urdf.xacro" />
+  <xacro:include filename="$(find xerbo_description)/urdf/imu.urdf.xacro" />
+  <xacro:include filename="$(find xerbo_description)/urdf/lidar.urdf.xacro" />
 </robot>
