Commit message: Updated URDF with BNO055 IMU physical mounting coord

File: src/xerbo_description/urdf/base.urdf.xacro (robot description, xacro)
@@ -1,4 +1,5 @@
 <?xml version="1.0"?>
 <robot xmlns:xacro="http://ros.org/wiki/xacro">
+  <!-- Top of base is z = 0.072-->
   <!-- Define robot constants -->
   <xacro:property name="wheel_separation" value="0.235"/>
@@ -11,9 +12,9 @@
     <inertial>
       <mass value="2" />
-      <origin xyz="0 0 0.0" />
+      <origin xyz="0 0 0" />
       <inertia ixx="0.01" ixy="0.0" ixz="0.0" iyy="0.01" iyz="0.0" izz="0.5" />
     </inertial>
     <visual>
-      <origin xyz=" 0 0 0.0308" rpy="0 0 0" />
+      <origin xyz="0 0 0.0308" rpy="0 0 0" />
       <geometry>
         <!-- "file://" syntax is compatible with both RVIZ and Gazebo -->

File: src/xerbo_description/urdf/imu.urdf.xacro (robot description, xacro)
@@ -1,8 +1,13 @@
 <?xml version="1.0"?>
 <robot xmlns:xacro="http://ros.org/wiki/xacro">
-  <xacro:property name="imu_x_size" value="0.04" />
-  <xacro:property name="imu_y_size" value="0.08" />
-  <xacro:property name="imu_z_size" value="0.02" />
+  <xacro:property name="imu_x_size" value="0.027" />
+  <xacro:property name="imu_y_size" value="0.02" />
+  <xacro:property name="imu_z_size" value="0.004" />
   <link name="imu_link">
+    <inertial>
+      <mass value="0.001"/>
+      <origin rpy="0 0 0" xyz="0 0 0"/>
+      <inertia ixx="0.0001" ixy="0" ixz="0" iyy="0.000001" iyz="0" izz="0.0001"/>
+    </inertial>
     <visual>
       <geometry>
@@ -15,10 +20,9 @@
       </geometry>
     </collision>
-    <xacro:box_inertia m="0.1" w="0.1" d="0.1" h="0.1"/>
   </link>
   <joint name="imu_joint" type="fixed">
     <parent link="base_link"/>
     <child link="imu_link"/>
-    <origin xyz="0 0 0.5"/>
+    <origin xyz="0 0 0.170475"/>
   </joint>
   <xacro:include filename="$(find xerbo_description)/urdf/imu.gazebo.urdf.xacro" />
