Commit message: Updated RPLIDAR mounted positioning and added mounting plates

File: src/xerbo_description/urdf/imu.urdf.xacro (robot description, xacro)
@@ -10,9 +10,4 @@
       <inertia ixx="0.0001" ixy="0" ixz="0" iyy="0.000001" iyz="0" izz="0.0001"/>
     </inertial>
-    <visual>
-      <geometry>
-        <box size="${imu_x_size} ${imu_y_size} ${imu_z_size}"/>
-      </geometry>
-    </visual>
     <collision>
       <geometry>
@@ -20,4 +15,12 @@
       </geometry>
     </collision>
+    <visual>
+      <geometry>
+        <box size="${imu_x_size} ${imu_y_size} ${imu_z_size}"/>
+      </geometry>
+      <material name="hunter-green">
+        <color rgba="255 87 51 1"/>
+      </material>
+    </visual>
   </link>
   <joint name="imu_joint" type="fixed">

File: src/xerbo_description/urdf/lidar.gazebo.urdf.xacro (robot description, xacro)
@@ -17,5 +17,5 @@
         <range>
           <min>0.120000</min>
-          <max>3.5</max>
+          <max>12.0</max>
           <resolution>0.015000</resolution>
         </range>

File: src/xerbo_description/urdf/lidar.urdf.xacro (robot description, xacro)
@@ -1,10 +1,10 @@
 <?xml version="1.0"?>
 <robot xmlns:xacro="http://ros.org/wiki/xacro">
-  <xacro:property name="lidar_radius" value="0.0508" />
-  <xacro:property name="lidar_length" value="0.0555" />
+  <xacro:property name="lidar_radius" value="0.035" />
+  <xacro:property name="lidar_length" value="0.0254" />
   <link name="lidar_link">
     <inertial>
       <origin xyz="0 0 0" rpy="0 0 0"/>
-      <mass value="0.125"/>
+      <mass value="0.17"/>
       <inertia ixx="0.001"  ixy="0"  ixz="0" iyy="0.001" iyz="0" izz="0.001" />
     </inertial>
@@ -20,4 +20,5 @@
         <cylinder radius="${lidar_radius}" length="${lidar_length}"/>
       </geometry>
+      <material name="black"/>
     </visual>
   </link>
@@ -25,5 +26,5 @@
     <parent link="base_link"/>
     <child link="lidar_link"/>
-    <origin xyz="0 0 0.25" rpy="0 0 0"/>
+    <origin xyz="0.115 0 0.10375" rpy="0 0 0"/>
   </joint>
   <xacro:include filename="$(find xerbo_description)/urdf/lidar.gazebo.urdf.xacro" />

File: src/xerbo_description/urdf/xerbo.urdf.xacro (robot description, xacro)
@@ -1,12 +1,6 @@
 <?xml version="1.0"?>
 <robot name="xerbo" xmlns:xacro="http://ros.org/wiki/xacro">
-  <xacro:macro name="box_inertia" params="m w h d">
-    <inertial>
-      <origin xyz="0 0 0" rpy="${pi/2} 0 ${pi/2}"/>
-      <mass value="${m}"/>
-      <inertia ixx="${(m/12) * (h*h + d*d)}" ixy="0.0" ixz="0.0" iyy="${(m/12) * (w*w + d*d)}" iyz="0.0" izz="${(m/12) * (w*w + h*h)}"/>
-    </inertial>
-  </xacro:macro>
   <xacro:include filename="$(find xerbo_description)/urdf/base.urdf.xacro" />
+  <xacro:include filename="$(find xerbo_description)/urdf/mounting-frame.urdf.xacro" />
   <xacro:include filename="$(find xerbo_description)/urdf/imu.urdf.xacro" />
   <xacro:include filename="$(find xerbo_description)/urdf/lidar.urdf.xacro" />
