Commit message: Changed wheel joints from continuous to fixed to resolve RViz error

File: src/xerbo_description/urdf/base.gazebo.urdf.xacro (robot description, xacro)
@@ -54,5 +54,5 @@
     <max_vel>1.0</max_vel>
   </gazebo>
-  <gazebo reference="front_caster">
+  <gazebo reference="front_caster_link">
     <mu1>0.0</mu1>
     <mu2>0.0</mu2>

File: src/xerbo_description/urdf/base.urdf.xacro (robot description, xacro)
@@ -47,9 +47,9 @@
   <joint name="base_joint" type="fixed">
     <origin xyz="0 0 0.017" rpy="0 0 0" />
-    <parent link="base_link"/>
-    <child link="base_footprint"/>
+    <parent link="base_footprint"/>
+    <child link="base_link"/>
   </joint>
   <!-- Wheels -->
-  <xacro:macro name="create_wheel" params="prefix y_offset wheel_radius wheel_width">">
+  <xacro:macro name="create_wheel" params="prefix y_offset">">
     <link name="${prefix}_link">
       <inertial>
@@ -71,5 +71,5 @@
       </collision>
     </link>
-    <joint name="${prefix}_joint" type="continuous">
+    <joint name="${prefix}_joint" type="fixed">
       <origin xyz="0 ${y_offset} 0.015" rpy="0 0 0" />
       <parent link="base_link"/>
@@ -78,7 +78,7 @@
     </joint>
   </xacro:macro>
-  <xacro:create_wheel prefix="drivewhl_l" y_offset="${wheel_separation / 2}" wheel_radius="${wheel_radius}" wheel_width="${wheel_width}"/>
-  <xacro:create_wheel prefix="drivewhl_r" y_offset="${wheel_separation / -2}" wheel_radius="${wheel_radius}" wheel_width="${wheel_width}"/>
-  <link name="front_caster">
+  <xacro:create_wheel prefix="drivewhl_l" y_offset="${wheel_separation / 2}" />
+  <xacro:create_wheel prefix="drivewhl_r" y_offset="${wheel_separation / -2}" />
+  <link name="front_caster_link">
     <inertial>
       <origin xyz="0 0 0" />
@@ -99,8 +99,8 @@
     </collision>
   </link>
-  <joint name="caster_joint" type="fixed">
+  <joint name="front_caster_joint" type="fixed">
     <origin xyz="0.13 0 0.0" rpy="0 0 0" />
     <parent link="base_link"/>
-    <child link="front_caster"/>
+    <child link="front_caster_link"/>
     <axis xyz="0 1 0" />
   </joint>

File: src/xerbo_description/urdf/imu.urdf.xacro (robot description, xacro)
@@ -20,5 +20,5 @@
       </geometry>
       <material name="hunter-green">
-        <color rgba="255 87 51 1"/>
+        <color rgba="1 0.34 0.2 1.0"/>
       </material>
     </visual>
